File: okay-mult.sch (KiCad schematic (older format))
At the start: 45 parts, among them J1 Conn_02x05_Odd_Even, J10 Conn_01x02_Female, J11 Conn_01x02_Female, J12 Conn_01x02_Male, J13 Conn_01x02_Male, J14 Thonkiconn, J15 Thonkiconn, J16 Thonkiconn, J17 Thonkiconn, J18 Conn_01x01_Female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

Commit message: Bigger fatter traces
Parts:
- J1: footprint Connector_PinSocket_2.54mm:PinSocket_2x05_P2.54mm_Vertical -> Connector_PinHeader_2.54mm:PinHeader_2x05_P2.54mm_Vertical
Changed lines of the file:
@@
 F 0 "J1" H 1500 7367 50  0000 C CNN
 F 1 "Conn_02x05_Odd_Even" H 1500 7276 50  0000 C CNN
-F 2 "Connector_PinSocket_2.54mm:PinSocket_2x05_P2.54mm_Vertical" H 1450 6950 50  0001 C CNN
+F 2 "Connector_PinHeader_2.54mm:PinHeader_2x05_P2.54mm_Vertical" H 1450 6950 50  0001 C CNN
 F 3 "~" H 1450 6950 50  0001 C CNN
 	1    1450 6950
