File: okay-multv2/okay-multv2.kicad_pcb (KiCad board)
At the start: 2 copper layers, 48.3 x 109.9 mm, 49 parts, among them J1 Thonkiconn, J10 Thonkiconn, J11 Thonkiconn, J12 Conn_02x05_Odd_Even, J2 Thonkiconn, J3 Thonkiconn, J4 Thonkiconn, J5 Thonkiconn, J6 Thonkiconn, J7 Thonkiconn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

Commit message: Update v2
Parts:
- added J13: Conn_02x05_Odd_Even, Connector_PinHeader_2.54mm:PinHeader_2x05_P2.54mm_Vertical, B.Cu at (156.0, 53.8)
- added J14: Conn_02x05_Odd_Even, Connector_PinHeader_2.54mm:PinHeader_2x05_P2.54mm_Vertical, B.Cu at (184.4, 53.8)
- added J15: Thonkiconn, Connector_Audio:RAF__Jack_3.5mm_QingPu_WQP-PJ398SM_Vertical_CircularHoles, F.Cu at (156.2, 37.5)
- added J16: Conn_02x05_Odd_Even, Connector_PinHeader_2.54mm:PinHeader_2x05_P2.54mm_Vertical, B.Cu at (156.0, 117.3)
- J1: value Thonkiconn -> Conn_02x05_Odd_Even; footprint Connector_Audio:RAF__Jack_3.5mm_QingPu_WQP-PJ398SM_Vertical_CircularHoles -> Connector_PinHeader_2.54mm:PinHeader_2x05_P2.54mm_Vertical; moved to B.Cu
- J12: moved to B.Cu
- moved R7 112.7 mm to (194.2, 39.4), turned to 180 degrees
- moved R4 103.4 mm to (184.3, 39.4)
- moved R5 102.5 mm to (184.5, 47.0)
- moved R6 102.0 mm to (193.9, 47.1), turned to 180 degrees
- moved R16 99.6 mm to (194.0, 62.2)
- moved R11 95.1 mm to (197.4, 105.5)
- moved C7 92.4 mm to (194.3, 43.2)
- moved R3 91.3 mm to (193.8, 111.0), turned to 90 degrees
- moved C6 89.5 mm to (184.6, 86.4), turned to 180 degrees
- moved C9 88.7 mm to (194.4, 108.0)
- moved R17 87.5 mm to (194.6, 90.3), turned to 180 degrees
- moved C10 87.1 mm to (184.5, 66.0), turned to 180 degrees
- moved R10 86.7 mm to (194.5, 105.5)
- moved J1 84.7 mm to (184.3, 117.3), turned to 270 degrees
- moved C4 83.7 mm to (184.3, 108.0), turned to 180 degrees
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Connections:
- J12 pad 3: Net-(J12-Pad3) -> GND
- J12 pad 5: Net-(J12-Pad3) -> GND
- J12 pad 7: Net-(J12-Pad3) -> GND
- J2 pad T: Net-(J2-PadT) -> Net-(J13-Pad2)
- J3 pad T: Net-(J3-PadT) -> Net-(J13-Pad4)
- J4 pad T: Net-(J4-PadT) -> Net-(J13-Pad6)
- J5 pad T: Net-(J5-PadT) -> Net-(J13-Pad8)
- J6 pad T: IN_B -> Net-(J13-Pad7)
- J6 pad TN: IN_A -> Net-(J13-Pad5)
- J7 pad T: Net-(J7-PadT) -> Net-(J16-Pad1)
- J8 pad T: Net-(J8-PadT) -> Net-(J16-Pad4)
- J9 pad T: Net-(J9-PadT) -> Net-(J16-Pad6)
- R11 pad 2: Net-(J11-PadT) -> /MIX_OUT
- R12 pad 1: Net-(D2-Pad1) -> /B_LED
- R13 pad 2: Net-(J7-PadT) -> /B1
- R14 pad 2: Net-(J8-PadT) -> /B2
- R15 pad 2: Net-(J9-PadT) -> /B3
- R16 pad 2: Net-(J10-PadT) -> /B4
- R17 pad 1: Net-(D5-Pad1) -> /MIX_LED
- R4 pad 1: Net-(J2-PadT) -> /A1
- R5 pad 1: Net-(J3-PadT) -> /A2
- R6 pad 1: Net-(J4-PadT) -> /A3
- R7 pad 1: Net-(J5-PadT) -> /A4
- R8 pad 1: Net-(D1-Pad1) -> /A_LED
Routing:
- net VEE: track 0.00 -> 104.7 mm, vias 0 -> 5
- net VCC: track 0.00 -> 103.3 mm, vias 0 -> 5
- net IN_A: track 0.00 -> 87.0 mm, vias 0 -> 3
- net IN_B: track 0.00 -> 69.5 mm
- net /B_LED: track 0.00 -> 44.9 mm, vias 0 -> 1
- net /A_LED: track 0.00 -> 30.5 mm
- net /A4: track 0.00 -> 19.2 mm
- net /A1: track 0.00 -> 19.1 mm, vias 0 -> 1
- net GND: track 0.00 -> 14.7 mm, vias 0 -> 11
- net /A3: track 0.00 -> 11.3 mm
- net /A2: track 0.00 -> 10.5 mm
- net Net-(D4-Pad1): track 0.00 -> 8.73 mm
- net Net-(D3-Pad2): track 0.00 -> 8.41 mm
- net Net-(R17-Pad2): track 0.00 -> 3.86 mm
- net Net-(R7-Pad2): track 0.00 -> 3.49 mm
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- added copper zone on GND, net GND
Other:
- copper layers 2 -> 4
- board text added: "~THE LINE~"
