File: okay-multv2/okay-multv2.sch (KiCad schematic (older format))
At the start: 49 parts, among them J1 Thonkiconn, J10 Thonkiconn, J11 Thonkiconn, J12 Conn_02x05_Odd_Even, J2 Thonkiconn, J3 Thonkiconn, J4 Thonkiconn, J5 Thonkiconn, J6 Thonkiconn, J7 Thonkiconn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

Commit message: Update v2
Parts:
- removed J1: Thonkiconn, Connector_Audio:RAF__Jack_3.5mm_QingPu_WQP-PJ398SM_Vertical_CircularHoles, symbol Connector:AudioJack2_SwitchT
- added J1, J13, J14, J16: Conn_02x05_Odd_Even, Connector_PinHeader_2.54mm:PinHeader_2x05_P2.54mm_Vertical, symbol Connector_Generic:Conn_02x05_Odd_Even
- added J15: Thonkiconn, Connector_Audio:RAF__Jack_3.5mm_QingPu_WQP-PJ398SM_Vertical_CircularHoles, symbol Connector:AudioJack2_SwitchT
Connections:
- net GND: now also J1.10 (Pin_10), J1.9 (Pin_9), J13.10 (Pin_10), J13.9 (Pin_9), J14.10 (Pin_10), J14.9 (Pin_9), J15.S, J16.10 (Pin_10), J16.9 (Pin_9)
- net IN_A: now also J14.5 (Pin_5); no longer J6.TN
- net IN_B: now also J14.7 (Pin_7); no longer J6.T
- net at J2.T: now also J13.2 (Pin_2); no longer R4.1
- net at J3.T: now also J13.4 (Pin_4); no longer R5.1
- net at J4.T: now also J13.6 (Pin_6); no longer R6.1
- net at J5.T: now also J13.8 (Pin_8); no longer R7.1
- net at J11.T: now also J16.2 (Pin_2); no longer R11.2
- net at J7.T: now also J16.1 (Pin_1); no longer R13.2
- net at J8.T: now also J16.4 (Pin_4); no longer R14.2
- net at J9.T: now also J16.6 (Pin_6); no longer R15.2
- net at J10.T: now also J16.8 (Pin_8); no longer R16.2
- net at D2.1 (KA): now also J13.3 (Pin_3); no longer R12.1
- net at D1.1 (KA): now also J13.1 (Pin_1); no longer R8.1
- net at D5.1 (KA): now also J16.3 (Pin_3); no longer R17.1
- new net: J13.7 (Pin_7), J6.T
- new net: J13.5 (Pin_5), J15.T, J6.TN
- new net A1: J14.2 (Pin_2), R4.1
- new net A2: J14.4 (Pin_4), R5.1
- new net A3: J14.6 (Pin_6), R6.1
- new net A4: J14.8 (Pin_8), R7.1
- new net A_LED: J14.1 (Pin_1), R8.1
- new net B1: J1.2 (Pin_2), R13.2
- new net B2: J1.4 (Pin_4), R14.2
- new net B3: J1.6 (Pin_6), R15.2
- new net B4: J1.8 (Pin_8), R16.2
- new net B_LED: J14.3 (Pin_3), R12.1
- new net MIX_LED: J1.3 (Pin_3), R17.1
- new net MIX_OUT: J1.1 (Pin_1), R11.2
Other:
- moved on the sheet: C1, C10, C11, C2, C3, C4, C5, C6, C7, C8, C9, D1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
